Commit message: Modified robots urdf

File: box_bot_description/robot/box_bot_v2.urdf (robot description, URDF)
Before this commit: robot box_bot, 12 links, 11 joints
Links:
- link chassis: geometry collision cylinder length=0.1 radius=0.05; visual cylinder length=0.1 radius=0.05
- link left_wheel: geometry collision cylinder length=0.01 radius=0.035; visual cylinder length=0.01 radius=0.035
- link right_wheel: geometry collision cylinder length=0.01 radius=0.035; visual cylinder length=0.01 radius=0.035
